File: estacao_metereologica_lora.kicad_sch (KiCad schematic)
At the start: 41 parts, among them IC1 E22-900M22S, J1 Font Conector, J10 PGM, J2 USB_B_Micro, J3 Batery Conector, J4 I2C_Con, J5 ADC_DAC Pins, J6 I2C_Con, J9 Display_I2C, Q1 FS8205A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

Commit message: Atualizando esquematico
Other:
- company: (none) -> Julio Nunes Avelar | Embarcações
- title: (none) -> Estação Metereologica LoRaWAN
Changed lines of the file:
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@@
 	(generator_version "8.0")
 	(paper "A4")
+	(title_block
+		(title "Estação Metereologica LoRaWAN")
+		(date "2024-03-24")
+		(rev "v1.0")
+		(company "Julio Nunes Avelar | Embarcações")
+	)
 	(junction
 		(at 176.53 83.82)

Commit message: Adicionando esquematico e componentes usados
Adicionando PDF do esquematico, footprints, simbolos e outras coisas
utilizadas no projeto
Other:
- title: Estação Metereologica LoRaWAN -> Estação Metereologica LoRaWAN | Colubris
Changed lines of the file:
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@@
 	(paper "A4")
 	(title_block
-		(title "Estação Metereologica LoRaWAN")
+		(title "Estação Metereologica LoRaWAN | Colubris")
 		(date "2024-03-24")
 		(rev "v1.0")
